File: gameport/gameport.sch (KiCad schematic (older format))
At the start: 38 parts, among them J1 Conn_01x10, J2 DB15_Female, J3 X, J4 Y, J5 B1, J6 B2, U1 LDL1117S50R, U2 TL072, U3 40106, U4 555, U5 555, U6 555

Commit message: Update schematic
Parts:
- removed U2: TL072, Package_DIP:DIP-8_W7.62mm, symbol Amplifier_Operational:TL072
- added C19, C20: 0.1uF, Capacitor_THT:C_Disc_D3.0mm_W1.6mm_P2.50mm, symbol Device:C_Small
- added R10, R11, R12, R13, R4, R5, R8, R9: 100k, Resistor_THT:R_Axial_DIN0207_L6.3mm_D2.5mm_P10.16mm_Horizontal, symbol Device:R
- added RV2: 10k, Potentiometer_THT:Potentiometer_Bourns_3296Y_Vertical, symbol Device:R_POT_TRIM
- added RV3: 22k, Potentiometer_THT:Potentiometer_Bourns_3296Y_Vertical, symbol Device:R_POT_TRIM
- added U2: TL074, Package_DIP:DIP-14_W7.62mm, symbol Amplifier_Operational:TL074
- C12, C13: value 10uF -> 1uF
- R14: renamed from R1; value 1k -> 10k
- R15: renamed from R2; value 1k -> 10k
- R3: renamed from R7; value 1k -> 22k
- R7: renamed from R8; value 1k -> 22k
- RV1: value 200k -> 100k
- gave numbers to parts that had none: 2
- renumbered R4 to R1, R5 to R2
Connections:
- net +12V: now also U2.4 (V+)
- net +5V: now also RV1.3, R10.2
- net -12V: now also U2.11 (V-)
- net GND: now also C19.2, C20.2, R11.2, R4.2, R8.2, U2.12 (+)
- net at J4.T: now also C20.1, R13.1
- net at C13.1, R7.1: now also U2.5 (+)
- net at C12.1, R3.1: now also U2.3 (+)
- net at J3.T: now also C19.1, R5.1
- new net: R5.2, RV3.1, U2.1
- new net: R4.1, RV3.2, RV3.3, U2.2 (-)
- new net: R8.1, RV2.2, RV2.3, U2.6 (-)
- new net: R9.2, RV2.1, U2.7
- new net: R10.1, R11.1, U2.10 (+)
- new net: R12.1, R13.2, U2.8
- new net: R12.2, R9.1, U2.9 (-)
- new net: U2.13 (-), U2.14
- no-connect marks 13 -> 12
Other:
- note added: "CLOCK SOURCE"
- note added: "Differential Amp - Unity Gain\nInverts response of Y direction"
- note added: "Gain = 1.1\nBoost 4.5V output to 5V"
- note added: "Gain = 1.22\nBoost 4V output to a full 5V"
- note added: "X DIRECTION"
- note added: "Y DIRECTION"
- moved on the sheet: C1, C10, C11, C12, C13, C14, C15, C16, C17, C18, C2, C3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

Commit message: Complete layout
Connections:
- net GND: now also U2.10 (+); no longer J2.12 (P12), U2.12 (+)
- net PWM_X: now reaches C18.1, R3.2, U5.3 (OUT)
- net PWM_Y: now reaches C17.1, R7.2, U6.3 (OUT)
- net at R4.1, RV3.2: now also RV3.1, U2.6 (-); no longer RV3.3, U2.2 (-)
- net at C12.1, R3.1: now also U2.5 (+); no longer U2.3 (+)
- net at C13.1, R7.1: now also U2.3 (+); no longer U2.5 (+)
- net at R8.1, RV2.2, RV2.3: now also U2.2 (-); no longer U2.6 (-)
- net at R9.2, RV2.1: now also U2.1; no longer U2.7
- net at R10.1, R11.1: now also U2.12 (+); no longer U2.10 (+)
- net at R12.1, R13.2: now also U2.14; no longer U2.8
- net at R12.2, R9.1: now also U2.13 (-); no longer U2.9 (-)
- new net: R5.2, RV3.3, U2.7
- new net: U2.8, U2.9 (-)
- no-connect marks 12 -> 13
Other:
- moved on the sheet: U2A, U2B, U2C, U2D
Changed lines of the file:
@@
 Wire Wire Line
 	5350 7100 5350 7200
-Wire Wire Line
-	1700 1750 1800 1750
-Wire Wire Line
-	1800 1850 1700 1850
-Wire Wire Line
-	1800 1750 1800 1850
-Wire Wire Line
-	1800 1750 1900 1750
-Connection ~ 1800 1750
 $Comp
 L power:GND #PWR08
@@
 L Amplifier_Operational:TL074 U2
 U 1 1 606D4B99
-P 8750 1900
-F 0 "U2" H 8750 2267 50  0000 C CNN
-F 1 "TL074" H 8750 2176 50  0000 C CNN
-F 2 "Package_DIP:DIP-14_W7.62mm" H 8700 2000 50  0001 C CNN
-F 3 "http://www.ti.com/lit/ds/symlink/tl071.pdf" H 8800 2100 50  0001 C CNN
-	1    8750 1900
+P 7150 4200
+F 0 "U2" H 7150 4567 50  0000 C CNN
+F 1 "TL074" H 7150 4476 50  0000 C CNN
+F 2 "Package_DIP:DIP-14_W7.62mm" H 7100 4300 50  0001 C CNN
+F 3 "http://www.ti.com/lit/ds/symlink/tl071.pdf" H 7200 4400 50  0001 C CNN
+	1    7150 4200
 	1    0    0    -1
 $EndComp
@@
 L Amplifier_Operational:TL074 U2
 U 4 1 606D9BCE
-P 10450 3250
-F 0 "U2" H 10450 2883 50  0000 C CNN
-F 1 "TL074" H 10450 2974 50  0000 C CNN
-F 2 "Package_DIP:DIP-14_W7.62mm" H 10400 3350 50  0001 C CNN
-F 3 "http://www.ti.com/lit/ds/symlink/tl071.pdf" H 10500 3450 50  0001 C CNN
-	4    10450 3250
+P 8800 4300
+F 0 "U2" H 8800 3933 50  0000 C CNN
+F 1 "TL074" H 8800 4024 50  0000 C CNN
+F 2 "Package_DIP:DIP-14_W7.62mm" H 8750 4400 50  0001 C CNN
+F 3 "http://www.ti.com/lit/ds/symlink/tl071.pdf" H 8850 4500 50  0001 C CNN
+	4    8800 4300
 	1    0    0    1
 $EndComp
@@
 L Amplifier_Operational:TL074 U2
 U 3 1 606D822F
-P 8800 4300
-F 0 "U2" H 8800 3933 50  0000 C CNN
-F 1 "TL074" H 8800 4024 50  0000 C CNN
-F 2 "Package_DIP:DIP-14_W7.62mm" H 8750 4400 50  0001 C CNN
-F 3 "http://www.ti.com/lit/ds/symlink/tl071.pdf" H 8850 4500 50  0001 C CNN
-	3    8800 4300
+P 10450 3250
+F 0 "U2" H 10450 3650 50  0000 C CNN
+F 1 "TL074" H 10450 3550 50  0000 C CNN
+F 2 "Package_DIP:DIP-14_W7.62mm" H 10400 3350 50  0001 C CNN
+F 3 "http://www.ti.com/lit/ds/symlink/tl071.pdf" H 10500 3450 50  0001 C CNN
+	3    10450 3250
 	1    0    0    1
 $EndComp
@@
 L Amplifier_Operational:TL074 U2
 U 2 1 606D67EC
-P 7150 4200
-F 0 "U2" H 7150 4567 50  0000 C CNN
-F 1 "TL074" H 7150 4476 50  0000 C CNN
-F 2 "Package_DIP:DIP-14_W7.62mm" H 7100 4300 50  0001 C CNN
-F 3 "http://www.ti.com/lit/ds/symlink/tl071.pdf" H 7200 4400 50  0001 C CNN
-	2    7150 4200
+P 8750 1900
+F 0 "U2" H 8750 2267 50  0000 C CNN
+F 1 "TL074" H 8750 2176 50  0000 C CNN
+F 2 "Package_DIP:DIP-14_W7.62mm" H 8700 2000 50  0001 C CNN
+F 3 "http://www.ti.com/lit/ds/symlink/tl071.pdf" H 8800 2100 50  0001 C CNN
+	2    8750 1900
 	1    0    0    -1
 $EndComp
@@
 F 3 "~" H 9050 2200 50  0001 C CNN
 	1    9050 2200
-	-1   0    0    -1
+	-1   0    0    1
 $EndComp
 Wire Wire Line
@@
 	9300 4300 9200 4300
 Connection ~ 9200 4300
+Wire Wire Line
+	1700 1750 1900 1750
+NoConn ~ 1700 1850
+Text Label 7200 1800 0    50   ~ 0
+PWM_X
+Text Label 5600 4100 0    50   ~ 0
+PWM_Y
 $EndSCHEMATC
