File: gameport/gameport.kicad_pcb (KiCad board)
At the start: 2 copper layers, 61 x 48.3 mm, 36 parts, among them J1 Conn_01x10, J2 DB15_Female, J3 X, J4 Y, J5 B1, J6 B2, U1 LDL1117S50R, U2 TL072, U3 40106, U4 555, U5 555, U6 555

Commit message: Complete layout
Parts:
- added C17: 0.1uF, Capacitor_THT:C_Disc_D3.0mm_W1.6mm_P2.50mm, F.Cu at (119.4, 78.7)
- added C18: 0.1uF, Capacitor_THT:C_Disc_D3.0mm_W1.6mm_P2.50mm, F.Cu at (119.4, 94.0)
- added C19: 0.1uF, Capacitor_THT:C_Disc_D3.0mm_W1.6mm_P2.50mm, F.Cu at (168.9, 97.8)
- added C20: 0.1uF, Capacitor_THT:C_Disc_D3.0mm_W1.6mm_P2.50mm, F.Cu at (168.9, 85.1)
- added R10: 100k, Resistor_THT:R_Axial_DIN0207_L6.3mm_D2.5mm_P10.16mm_Horizontal, F.Cu at (158.8, 92.7)
- added R11: 100k, Resistor_THT:R_Axial_DIN0207_L6.3mm_D2.5mm_P10.16mm_Horizontal, F.Cu at (158.8, 95.2)
- added R12: 100k, Resistor_THT:R_Axial_DIN0207_L6.3mm_D2.5mm_P10.16mm_Horizontal, F.Cu at (158.8, 90.2)
- added R13: 100k, Resistor_THT:R_Axial_DIN0207_L6.3mm_D2.5mm_P10.16mm_Horizontal, F.Cu at (168.9, 87.6)
- added R4: 100k, Resistor_THT:R_Axial_DIN0207_L6.3mm_D2.5mm_P10.16mm_Horizontal, F.Cu at (138.4, 105.4)
- added R5: 100k, Resistor_THT:R_Axial_DIN0207_L6.3mm_D2.5mm_P10.16mm_Horizontal, F.Cu at (168.9, 100.3)
- added R8: 100k, Resistor_THT:R_Axial_DIN0207_L6.3mm_D2.5mm_P10.16mm_Horizontal, F.Cu at (138.4, 85.1)
- added R9: 100k, Resistor_THT:R_Axial_DIN0207_L6.3mm_D2.5mm_P10.16mm_Horizontal, F.Cu at (161.3, 85.1)
- added RV2: 10k, Potentiometer_THT:Potentiometer_Bourns_3296Y_Vertical, F.Cu at (144.8, 87.6)
- added RV3: 22k, Potentiometer_THT:Potentiometer_Bourns_3296Y_Vertical, F.Cu at (139.7, 102.9)
- C12, C13: value 10uF -> 1uF
- R14: renamed from R1; value 1k -> 10k
- R15: renamed from R2; value 1k -> 10k
- R3: renamed from R7; value 1k -> 22k
- R7: renamed from R8; value 1k -> 22k
- RV1: value 200k -> 100k
- U2: value TL072 -> TL074; footprint Package_DIP:DIP-8_W7.62mm -> Package_DIP:DIP-14_W7.62mm
- moved C2 50.8 mm to (179.1, 71.1), turned to 0 degrees
- moved C1 43.4 mm to (179.1, 77.3), turned to 0 degrees
- moved U1 38.2 mm to (173.4, 74.3), turned to 90 degrees
- moved C4 21.6 mm to (161.3, 97.8), turned to 180 degrees
- moved J1 18.0 mm to (180.3, 99.1)
- moved C3 8.99 mm to (146.1, 94.0), turned to 270 degrees
- moved J3 8.89 mm to (152.4, 77.5)
- moved J4 8.89 mm to (161.3, 77.5)
- moved C13 8.18 mm to (137.2, 93.2)
- moved C12 5.93 mm to (142.2, 97.2)
- moved U2 4.58 mm to (148.6, 87.6), turned to 0 degrees
- moved U3 1.27 mm to (135.9, 64.8)
- moved C5 1.27 mm to (146.1, 64.8)
- moved R14 1.27 mm to (146.1, 80.0)
- renumbered R4 to R1, R5 to R2
Connections:
- net Net-(R7-Pad2) renamed /PWM_X
- net Net-(R8-Pad2) renamed /PWM_Y
- J2 pad 12: GND -> Net-(J2-Pad12)
- J3 pad T: Net-(J3-PadT) -> Net-(C19-Pad1)
- J4 pad T: Net-(J4-PadT) -> Net-(C20-Pad1)
- RV1 pad 3: Net-(RV1-Pad3) -> +5V
- U2 pad 1: Net-(J4-PadT) -> Net-(R9-Pad2)
- U2 pad 2: Net-(J4-PadT) -> Net-(R8-Pad1)
- U2 pad 4: -12V -> +12V
- U2 pad 6: Net-(J3-PadT) -> Net-(R4-Pad1)
- U2 pad 7: Net-(J3-PadT) -> Net-(R5-Pad2)
- U2 pad 8: +12V -> Net-(U2-Pad8)
Routing:
- net +12V: track 30.3 -> 71.6 mm
- net Net-(C19-Pad1): track 0.00 -> 29.7 mm
- net Net-(R12-Pad2): track 0.00 -> 23.5 mm
- net Net-(J3-PadT): track 22.5 -> 0.00 mm
- net Net-(R5-Pad2): track 0.00 -> 15.0 mm
- net Net-(C20-Pad1): track 0.00 -> 13.3 mm
- net Net-(R4-Pad1): track 0.00 -> 13.0 mm
- net Net-(R8-Pad1): track 0.00 -> 13.0 mm
- net Net-(J4-PadT): track 10.2 -> 0.00 mm
- net Net-(J6-PadT): track 8.67 -> 18.6 mm
- net Net-(C13-Pad1): track 20.0 -> 28.3 mm
- net Net-(R9-Pad2): track 0.00 -> 7.40 mm
- net Net-(R12-Pad1): track 0.00 -> 5.08 mm
- net Net-(R10-Pad1): track 0.00 -> 5.08 mm
- net Net-(C12-Pad1): track 13.2 -> 18.1 mm
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Other:
- board size 61 x 48.3 mm -> 78.7 x 48.3 mm
- board text added: "Apr 2021 v0.1"
- board text added: "github.com/mprosk/gameport"
- board text removed: "Max Proskauer Mar 2021 v0.1"

Commit message: Update to Kicad6. Use kosmo-lib submodule
Connections:
- net /~B1 renamed /~{B1}
- net /~B2 renamed /~{B2}
Other:
- net class Default removed
- net class Power removed
