File: faceplate/gameport_faceplate.kicad_pcb (KiCad board)
At the start: 2 copper layers, 25 x 200 mm, 5 parts

Commit message: Update to Kicad6. Use kosmo-lib submodule
Other:
- net class Default removed
